File: UV_sensor/design/schemat1.sch (EAGLE design)
At the start: 13 parts, among them U1 MCP1703-3302E/CB

Commit message: update
Parts:
- removed C6: 1u, rcl:CPOL-EUSMCA
- removed CN2: (no value), adafruit:DCBARRELSMT
- removed U$1: UV-SENSOR-ML8511, diy-modules:UV-SENSOR-ML8511
- added C1: 47u, rcl:CPOL-EUCT3528
- added IC1: MCP1703CB, linear:MCP1703CB
- added JP1: (no value), pinhead:PINHD-1X2
- added JP2: (no value), pinhead:PINHD-1X4/90
- added R3: 1k, rcl:R-EU_R0805
- added R4: 100k, rcl:R-EU_R0805
- added R5: 230k, rcl:R-EU_R0805
- added R6: 10k, rcl:R-EU_R0805
- C4: device rcl:CPOL-EUSMCD -> rcl:CPOL-EUCT3528
- C5: value 47u -> 1u; device rcl:CPOL-EUSMCD -> rcl:CPOL-EUCT3216
- LED1: device adafruit:LEDCHIPLED_0805 -> eagle-ltspice:LED_E
- R1: value 10k -> 65R
- R2: value 65R -> 0R
- U1: value MCP1703-3302E/CB -> UV-SENSOR-ML8511; device _hhn_MCP1703:MCP1703-3302E/CB -> diy-modules:UV-SENSOR-ML8511
Connections:
- new net N$1: R5.1, U1.OUT
- new net N$3: MDL1.GPIO0, R2.2
- new net N$5: MDL1.GPIO15, R3.2
- net +3V3: now also C3.1, IC1.VO, R6.2, U1.3V3, U1.EN, U1.VIN; no longer C2.1, R1.2, U$1.3V3, U$1.EN, U$1.VIN, U1.VO
- net ADC: now also R4.2, R5.2; no longer U$1.OUT
- net GND: now also C1.-, IC1.GND, JP1.1, JP2.4, R1.1, R3.1, R4.1; no longer C6.-, CN2.GND, CN2.GNDBREAK, U$1.GND
- net N$2: now also R1.2; no longer R2.2
- net RESET: now also C5.+, R6.1; no longer C6.+, R1.1
- net RX: now also JP2.2, MDL1.TXD; no longer MDL1.RXD
- net TX: now also JP2.3, MDL1.RXD; no longer MDL1.TXD
- net VIN: now also C1.+, C2.1, IC1.VI, JP1.2, JP2.1; no longer C3.1, C5.+, CN2.PWR, U1.VI
Other:
- moved on the sheet: C2, C3, C4, C5, LED1, MDL1, R1, R2, S1
